File: robot/robot.sch (EAGLE design)
At the start: 12 parts, among them Q1 MOSFET-NCHANNELBSS138

Commit message: Cleaning up the pcb
Changed lines of the file:
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@@
 <wire x1="-27.94" y1="-5.08" x2="-27.94" y2="-2.54" width="0.1524" layer="91"/>
 <junction x="-27.94" y="-2.54"/>
+<label x="-35.56" y="0" size="1.778" layer="95"/>
 </segment>
 <segment>
@@
 <junction x="-25.4" y="-66.04"/>
 <pinref part="GND7" gate="1" pin="GND"/>
+<junction x="-25.4" y="-63.5"/>
 </segment>
 <segment>
